File: conductivity_sensor.kicad_pcb (KiCad board)
At the start: 2 copper layers, 76.2 x 76.2 mm, 29 parts, among them J1 Screw_Terminal_01x04, U1 MCP6024, U2 MAX4619, U3 MAX4619

Commit message: first version
Parts:
- added C10: C_X7R, passives:C_TH_CERAMIC_RADIAL_100mil, F.Cu at (113.7, 142.2)
- added U4: MCP9700A, actives:TO-92, B.Cu at (112.4, 139.1)
- moved R1 29.9 mm to (134.9, 139.7), turned to 0 degrees
- moved MK_2 18.4 mm to (135.3, 121.3)
- moved C4 17.4 mm to (159.4, 108.0), turned to 270 degrees
- moved C9 16.9 mm to (148.6, 121.2)
- moved R4 13.6 mm to (141.0, 111.8), turned to 180 degrees
- moved R3 9.71 mm to (144.8, 109.9), turned to 90 degrees
- moved U1 5.84 mm to (156.2, 114.9)
- moved C8 5.04 mm to (159.4, 102.2)
- moved D2 3.30 mm to (144.1, 123.2)
Routing:
- net Net-(A1-Pad20): track 0.00 -> 42.5 mm
- net Net-(C9-Pad1): track 71.8 -> 58.0 mm
- net Net-(U1-Pad1): track 51.2 -> 37.6 mm, vias 1 -> 0
- net Net-(R3-Pad1): track 21.9 -> 8.41 mm
- net Net-(D2-Pad2): track 10.1 -> 21.2 mm
- net Net-(R5-Pad1): track 20.9 -> 31.3 mm
- net /PEAK: track 98.7 -> 109.1 mm
- net VREF: track 148.2 -> 158.2 mm
- net Net-(C8-Pad1): track 45.1 -> 53.1 mm, vias 0 -> 1
- net Net-(MK_2-Pad1): track 31.2 -> 28.1 mm
- net Net-(C8-Pad2): track 25.2 -> 27.8 mm, vias 0 -> 1
- net VCC: track 174.2 -> 176.0 mm, vias 6 -> 5
- net Net-(R_GAIN1-Pad2): track 6.92 -> 5.80 mm
Other:
- board text added: "- tx rx +5"
- board text added: "conductivity sensor umn bbe - dfuruta rev 1 march 2018"
